File: v1/hardware/midi-looper/midi-looper.sch (KiCad schematic (older format))
At the start: 29 parts, among them J1 SW1, J2 SW2, J3 SW3, J4 Batt IN, J5 SSD1306 SPI, J6 MIDI OUT 1 -Y:M5 R:M4, J7 MIDI OUT 2 -Y:M5 R:M4, J8 MIDI OUT 3 -Y:M5 R:M4, J9 Rot. Enc. Bk/Or:GND - Re:A - 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, U1 6N138, U2 Teensy3.2_breadboard_friendly, U3 6N138, U4 6N138

Commit message: Updated PCB and schem
Parts:
- added J10: Conn_01x05_Female, Connector_JST:JST_PH_B5B-PH-K_1x05_P2.00mm_Vertical, symbol Connector:Conn_01x05_Female
- added J11: MIDI IN 1 - Bk:M5 R:M4, Connector_JST:JST_XH_B2B-XH-A_1x02_P2.50mm_Vertical, symbol Connector:Conn_01x02_Female
- added J12: MIDI IN 2 - Bk:M5 R:M4, Connector_JST:JST_XH_B2B-XH-A_1x02_P2.50mm_Vertical, symbol Connector:Conn_01x02_Female
- added J13: MIDI IN 3 - Bk:M5 R:M4, Connector_JST:JST_XH_B2B-XH-A_1x02_P2.50mm_Vertical, symbol Connector:Conn_01x02_Female
- added SW1: Rotary_Encoder_Switch, Rotary_Encoder:RotaryEncoder_Alps_EC11E-Switch_Vertical_H20mm_CircularMountingHoles, symbol Device:Rotary_Encoder_Switch
- J1, J2, J3: footprint Connector_JST:JST_EH_B2B-EH-A_1x02_P2.50mm_Vertical -> Connector_JST:JST_XH_B2B-XH-A_1x02_P2.50mm_Vertical
- J5: footprint Connector_JST:JST_EH_B7B-EH-A_1x07_P2.50mm_Vertical -> Connector_PinHeader_2.54mm:PinHeader_1x07_P2.54mm_Vertical
- J6, J7, J8: footprint Connector_JST:JST_EH_B3B-EH-A_1x03_P2.50mm_Vertical -> Connector_JST:JST_PH_B3B-PH-K_1x03_P2.00mm_Vertical
- J9: footprint Connector_JST:JST_EH_B5B-EH-A_1x05_P2.50mm_Vertical -> Connector_JST:JST_PH_B5B-PH-K_1x05_P2.00mm_Vertical
Connections:
- net at D1.1 (K), U1.2 (C1): now also J11.2 (Pin_2)
- net at D1.2 (A), U1.3 (C2): now also J11.1 (Pin_1)
- net at D2.1 (K), U3.2 (C1): now also J12.2 (Pin_2)
- net at D2.2 (A), U3.3 (C2): now also J12.1 (Pin_1)
- net at D3.1 (K), U4.2 (C1): now also J13.2 (Pin_2)
- net at D3.2 (A), U4.3 (C2): now also J13.1 (Pin_1)
- new net: J10.4 (Pin_4), SW1.A
- new net: J10.3 (Pin_3), SW1.B
- new net: J10.1 (Pin_1), J10.5 (Pin_5), SW1.C, SW1.S2
- new net: J10.2 (Pin_2), SW1.S1
Changed lines of the file:
@@
 F 0 "J5" V 5365 3230 50  0000 C CNN
 F 1 "SSD1306 SPI" V 5274 3230 50  0000 C CNN
-F 2 "Connector_JST:JST_EH_B7B-EH-A_1x07_P2.50mm_Vertical" H 5200 3250 50  0001 C CNN
+F 2 "Connector_PinHeader_2.54mm:PinHeader_1x07_P2.54mm_Vertical" H 5200 3250 50  0001 C CNN
 F 3 "~" H 5200 3250 50  0001 C CNN
 	1    5200 3250
@@
 F 0 "J6" V 7488 1212 50  0000 R CNN
 F 1 "MIDI OUT 1 -Y:M5 R:M4" V 7397 1212 50  0000 R CNN
-F 2 "Connector_JST:JST_EH_B3B-EH-A_1x03_P2.50mm_Vertical" H 7550 1400 50  0001 C CNN
+F 2 "Connector_JST:JST_PH_B3B-PH-K_1x03_P2.00mm_Vertical" H 7550 1400 50  0001 C CNN
 F 3 "~" H 7550 1400 50  0001 C CNN
 	1    7550 1400
@@
 F 0 "J7" V 8438 1212 50  0000 R CNN
 F 1 "MIDI OUT 2 -Y:M5 R:M4" V 8347 1212 50  0000 R CNN
-F 2 "Connector_JST:JST_EH_B3B-EH-A_1x03_P2.50mm_Vertical" H 8500 1400 50  0001 C CNN
+F 2 "Connector_JST:JST_PH_B3B-PH-K_1x03_P2.00mm_Vertical" H 8500 1400 50  0001 C CNN
 F 3 "~" H 8500 1400 50  0001 C CNN
 	1    8500 1400
@@
 F 0 "J8" V 9388 1212 50  0000 R CNN
 F 1 "MIDI OUT 3 -Y:M5 R:M4" V 9297 1212 50  0000 R CNN
-F 2 "Connector_JST:JST_EH_B3B-EH-A_1x03_P2.50mm_Vertical" H 9450 1400 50  0001 C CNN
+F 2 "Connector_JST:JST_PH_B3B-PH-K_1x03_P2.00mm_Vertical" H 9450 1400 50  0001 C CNN
 F 3 "~" H 9450 1400 50  0001 C CNN
 	1    9450 1400
@@
 F 0 "J1" V 2888 2862 50  0000 R CNN
 F 1 "SW1" V 2797 2862 50  0000 R CNN
-F 2 "Connector_JST:JST_EH_B2B-EH-A_1x02_P2.50mm_Vertical" H 2950 3050 50  0001 C CNN
+F 2 "Connector_JST:JST_XH_B2B-XH-A_1x02_P2.50mm_Vertical" H 2950 3050 50  0001 C CNN
 F 3 "~" H 2950 3050 50  0001 C CNN
 	1    2950 3050
@@
 F 0 "J2" V 3288 2862 50  0000 R CNN
 F 1 "SW2" V 3197 2862 50  0000 R CNN
-F 2 "Connector_JST:JST_EH_B2B-EH-A_1x02_P2.50mm_Vertical" H 3350 3050 50  0001 C CNN
+F 2 "Connector_JST:JST_XH_B2B-XH-A_1x02_P2.50mm_Vertical" H 3350 3050 50  0001 C CNN
 F 3 "~" H 3350 3050 50  0001 C CNN
 	1    3350 3050
@@
 F 0 "J3" V 3638 2862 50  0000 R CNN
 F 1 "SW3" V 3547 2862 50  0000 R CNN
-F 2 "Connector_JST:JST_EH_B2B-EH-A_1x02_P2.50mm_Vertical" H 3700 3050 50  0001 C CNN
+F 2 "Connector_JST:JST_XH_B2B-XH-A_1x02_P2.50mm_Vertical" H 3700 3050 50  0001 C CNN
 F 3 "~" H 3700 3050 50  0001 C CNN
 	1    3700 3050
@@
 F 0 "J9" H 2692 3875 50  0000 C CNN
 F 1 "Rot. Enc. Bk/Or:GND - Re:A - Wh:B - Ye:SW" H 2692 3966 50  0000 C CNN
-F 2 "Connector_JST:JST_EH_B5B-EH-A_1x05_P2.50mm_Vertical" H 2800 4300 50  0001 C CNN
+F 2 "Connector_JST:JST_PH_B5B-PH-K_1x05_P2.00mm_Vertical" H 2800 4300 50  0001 C CNN
 F 3 "~" H 2800 4300 50  0001 C CNN
 	1    2800 4300
@@
 NoConn ~ 3600 5950
 NoConn ~ 3800 5950
+$Comp
+L Device:Rotary_Encoder_Switch SW1
+U 1 1 61C4AB4F
+P 1350 3800
+F 0 "SW1" H 1350 3433 50  0000 C CNN
+F 1 "Rotary_Encoder_Switch" H 1350 3524 50  0000 C CNN
+F 2 "Rotary_Encoder:RotaryEncoder_Alps_EC11E-Switch_Vertical_H20mm_CircularMountingHoles" H 1200 3960 50  0001 C CNN
+F 3 "~" H 1350 4060 50  0001 C CNN
+	1    1350 3800
+	-1   0    0    1
+$EndComp
+$Comp
+L Connector:Conn_01x05_Female J10
+U 1 1 61C4BD22
+P 2250 3600
+F 0 "J10" H 2278 3626 50  0000 L CNN
+F 1 "Conn_01x05_Female" H 2278 3535 50  0000 L CNN
+F 2 "Connector_JST:JST_PH_B5B-PH-K_1x05_P2.00mm_Vertical" H 2250 3600 50  0001 C CNN
+F 3 "~" H 2250 3600 50  0001 C CNN
+	1    2250 3600
+	1    0    0    -1
+$EndComp
+Wire Wire Line
+	2050 3400 2000 3400
+Wire Wire Line
+	1050 3400 1050 3700
+Wire Wire Line
+	2050 3800 2000 3800
+Wire Wire Line
+	1650 3900 1950 3900
+Wire Wire Line
+	1950 3900 1950 3700
+Wire Wire Line
+	1950 3700 2050 3700
+Wire Wire Line
+	1650 3700 1900 3700
+Wire Wire Line
+	1900 3700 1900 3600
+Wire Wire Line
+	1900 3600 2050 3600
+Wire Wire Line
+	2050 3500 850  3500
+Wire Wire Line
+	850  3500 850  3900
+Wire Wire Line
+	850  3900 1050 3900
+$Comp
+L Connector:Conn_01x02_Female J11
+U 1 1 61B7D2E3
+P 3950 1100
+F 0 "J11" V 3888 912 50  0000 R CNN
+F 1 "MIDI IN 1 - Bk:M5 R:M4" V 3797 912 50  0000 R CNN
+F 2 "Connector_JST:JST_XH_B2B-XH-A_1x02_P2.50mm_Vertical" H 3950 1100 50  0001 C CNN
+F 3 "~" H 3950 1100 50  0001 C CNN
+	1    3950 1100
+	0    -1   -1   0
+$EndComp
+$Comp
+L Connector:Conn_01x02_Female J12
+U 1 1 61B7EA12
+P 4900 1100
+F 0 "J12" V 4838 912 50  0000 R CNN
+F 1 "MIDI IN 2 - Bk:M5 R:M4" V 4747 912 50  0000 R CNN
+F 2 "Connector_JST:JST_XH_B2B-XH-A_1x02_P2.50mm_Vertical" H 4900 1100 50  0001 C CNN
+F 3 "~" H 4900 1100 50  0001 C CNN
+	1    4900 1100
+	0    -1   -1   0
+$EndComp
+$Comp
+L Connector:Conn_01x02_Female J13
+U 1 1 61B81B76
+P 5900 1100
+F 0 "J13" V 5838 912 50  0000 R CNN
+F 1 "MIDI IN 3 - Bk:M5 R:M4" V 5747 912 50  0000 R CNN
+F 2 "Connector_JST:JST_XH_B2B-XH-A_1x02_P2.50mm_Vertical" H 5900 1100 50  0001 C CNN
+F 3 "~" H 5900 1100 50  0001 C CNN
+	1    5900 1100
+	0    -1   -1   0
+$EndComp
+Wire Wire Line
+	3950 1300 3850 1300
+Wire Wire Line
+	3850 1300 3850 1650
+Connection ~ 3850 1650
+Wire Wire Line
+	4050 1300 4150 1300
+Wire Wire Line
+	4150 1300 4150 1650
+Connection ~ 4150 1650
+Wire Wire Line
+	4900 1300 4900 1400
+Wire Wire Line
+	4900 1400 4800 1400
+Wire Wire Line
+	4800 1400 4800 1650
+Connection ~ 4800 1650
+Wire Wire Line
+	5000 1300 5100 1300
+Wire Wire Line
+	5100 1300 5100 1650
+Connection ~ 5100 1650
+Wire Wire Line
+	5900 1300 5800 1300
+Wire Wire Line
+	5800 1300 5800 1650
+Connection ~ 5800 1650
+Wire Wire Line
+	6000 1300 6100 1300
+Wire Wire Line
+	6100 1300 6100 1650
+Connection ~ 6100 1650
+Wire Wire Line
+	2000 3400 2000 3800
+Connection ~ 2000 3400
+Wire Wire Line
+	2000 3400 1050 3400
+Connection ~ 2000 3800
+Wire Wire Line
+	2000 3800 1650 3800
 $EndSCHEMATC
